Commit message: added camera

File: src/arduinobot_description/urdf/arduinobot.urdf.xacro (robot description, xacro)
@@ -56,7 +56,7 @@
     </joint>
     <link name="rgb_camera">
-        <xacro:default_inertial mass="0.1"/>
-        <visual>
-            <origin rpy="0 1.57 0" xyz="0 -0.125 0.125"/>
+        <xacro:default_inertial mass="0.001"/>
+        <visual>
+            <origin rpy="-1.57 0 -1.57" xyz="-0.1 0.125 0.15"/>
             <geometry>
                 <mesh filename="package://arduinobot_description/meshes/pi_camera.STL" scale="0.01 0.01 0.01"/>
@@ -64,10 +64,34 @@
         </visual>
         <collision>
-            <origin rpy="0 0 0" xyz="-0.5 -0.5 0"/>
-            <geometry>
-                <mesh filename="package://arduinobot_description/meshes/basement.STL" scale="0.01 0.01 0.01"/>
-            </geometry>
-        </collision>
-    </link>
+            <origin rpy="-1.57 0 -1.57" xyz="-0.1 0.125 0.15"/>
+            <geometry>
+                <mesh filename="package://arduinobot_description/meshes/pi_camera.STL" scale="0.01 0.01 0.01"/>
+            </geometry>
+        </collision>
+    </link>
+    <gazebo>
+        <sensor type="camera" name="camera1">
+            <update_rate>30</update_rate>
+            <visualize>true</visualize>
+            <camera name="head">
+              <horizontal_fov>1.15</horizontal_fov>
+              <vertical_fov>0.71</vertical_fov>
+              <image>
+                <width>2304</width>
+                <height>1296</height>
+                <format>R8G8B8</format>
+              </image>
+            </camera>
+            <plugin name="plugin_name" filename="libgazebo_ros_camera.so">
+                <ros>
+                  <remapping>image_raw:=image_raw</remapping>
+                  <remapping>camera_info:=camera_info</remapping>
+                </ros>
+                <camera_name>rgb_camera</camera_name>
+                <frame_name>rgb_camera</frame_name>
+                <hack_baseline>0.2</hack_baseline>
+              </plugin>
+          </sensor>
+    </gazebo>
     <joint name="rgb_camera_joint" type="fixed">
         <parent link="base_link"/>

Commit message: implemented controller launch file

File: src/arduinobot_description/urdf/arduinobot.urdf.xacro (robot description, xacro)
@@ -1,4 +1,6 @@
 <?xml version = "1.0"?>
 <robot xmlns:xacro="http://www.ros.org/wiki/xacro" name="arduinobot">
+    <xacro:include filename="$(find arduinobot_description)/urdf/arduinobot_gazebo.xacro"/>
+    <xacro:include filename="$(find arduinobot_description)/urdf/arduinobot_ros2_control.xacro"/>
     <xacro:property name="PI" value="3.14159"/>
     <xacro:property name="effort" value="30"/>
@@ -11,4 +13,13 @@
                     izz="1.0"/>
         </inertial>
+    </xacro:macro>
+    <xacro:macro name="default_transmission" params = "number">
+        <transmission name="transmission_${number}">
+            <plugin>transmission_interface/SimpleTransmission</plugin>
+            <actuator name="motor_${number}" role = "actuator1"/>
+            <joint name="joint_${number}" rolw="joint1">
+                <mechanical_reduction>1.0</mechanical_reduction>
+            </joint>
+        </transmission>
     </xacro:macro>
     <link name="world"/>
@@ -209,3 +220,7 @@
         <limit lower="0" upper="${PI/2}" effort="${effort}" velocity="${velocity}"/>
     </joint>
+    <xacro:default_transmission number="1"/>
+    <xacro:default_transmission number="2"/>
+    <xacro:default_transmission number="3"/>
+    <xacro:default_transmission number="4"/>
 </robot>

Commit message: debug

File: src/arduinobot_description/urdf/arduinobot.urdf.xacro (robot description, xacro)
@@ -1,4 +1,5 @@
 <?xml version = "1.0"?>
 <robot xmlns:xacro="http://www.ros.org/wiki/xacro" name="arduinobot">
+    <xacro:arg name="is_sim" default = "true"/>
     <xacro:include filename="$(find arduinobot_description)/urdf/arduinobot_gazebo.xacro"/>
     <xacro:include filename="$(find arduinobot_description)/urdf/arduinobot_ros2_control.xacro"/>

File: src/arduinobot_description/urdf/arduinobot_ros2_control.xacro (robot description, xacro)
@@ -1,6 +1,26 @@
 <?xml version="1.0"?>
 <robot xmlns:xacro="http://www.ros.org/wiki/xacro" name="aduinobot">
-    <xacro:property name="PI" value="3.14159"/>
     <ros2_control name="RobotSystem" type="system">
+        <xacro:property name="PI" value="3.14159"/>
+        <xacro:if value="$(arg is_sim)">
+            <hardware>
+                <plugin>gazebo_ros2_control/GazeboSystem</plugin>
+            </hardware>
+            <joint name="joint_5">
+                <param name="mimic">joint_4</param>
+                <paraam name="multiplier">-1</paraam>
+                <command_interface name="position">
+                    <param name="min">0.0</param>
+                    <param name="max">${PI/2}</param>
+                </command_interface>
+                <state_interface name="position"/>
+            </joint>
+        </xacro:if>
+        <xacro:unless value="$(arg is_sim)">
+            <hardware>
+                <plugin>arduinobot_controller/ArduinobotInterface</plugin>
+                <param name = "port">/dev/ttyACM0</param>
+            </hardware>
+        </xacro:unless>
         <hardware>
             <plugin>gazebo_ros2_control/GazeboSystem</plugin>
@@ -34,13 +54,4 @@
             <state_interface name="position"/>
         </joint>
-        <joint name="joint_5">
-            <param name="mimic">joint_4</param>
-            <paraam name="multiplier">-1</paraam>
-            <command_interface name="position">
-                <param name="min">0.0</param>
-                <param name="max">${PI/2}</param>
-            </command_interface>
-            <state_interface name="position"/>
-        </joint>
     </ros2_control>
 </robot>
