Commit message: fix the xacro bug, need space behind because it's separating the xacro and the rest of the command otherwise it would be considered a part of the path which is not correct.

File: src/arduinobot_description/urdf/arduinobot_gazebo.xacro (robot description, xacro)
@@ -1,10 +1,11 @@
 <?xml version="1.0"?>
-<robot xmlns:xacro="http://www.ros.org/wiki/xacro" name="aduinobot">
+<robot xmlns:xacro="http://www.ros.org/wiki/xacro" name="arduinobot">
+    <!-- Gazebo ros2_control plugin -->
     <gazebo>
-        <plugin filename="libgazebo_ros2_control.so" name="gazebo_ros2_control">
-            <robot_param>robot_description</robot_param>
-            <robot_param_node>robot_state_publisher</robot_param_node>
-            <parameters>$(find arduinobot_controller)/config/arduinobot_controllers.yaml</parameters>
-        </plugin>
+      <plugin filename="libgazebo_ros2_control.so" name="gazebo_ros2_control">
+        <robot_param>robot_description</robot_param>
+        <robot_param_node>robot_state_publisher</robot_param_node>
+        <parameters>$(find arduinobot_controller)/config/arduinobot_controllers.yaml</parameters>
+      </plugin>
     </gazebo>
 </robot>

File: src/arduinobot_description/urdf/arduinobot_ros2_control.xacro (robot description, xacro)
@@ -1,6 +1,7 @@
 <?xml version="1.0"?>
-<robot xmlns:xacro="http://www.ros.org/wiki/xacro" name="aduinobot">
+<robot xmlns:xacro="http://www.ros.org/wiki/xacro" name="arduinobot">
     <ros2_control name="RobotSystem" type="system">
-        <xacro:property name="PI" value="3.14159"/>
+        <xacro:property name="PI" value="3.14159265359" />
+        <!-- ros2_control Gazebo -->
         <xacro:if value="$(arg is_sim)">
             <hardware>
@@ -9,25 +10,22 @@
             <joint name="joint_5">
                 <param name="mimic">joint_4</param>
-                <paraam name="multiplier">-1</paraam>
+                <param name="multiplier">-1</param>
                 <command_interface name="position">
-                    <param name="min">0.0</param>
-                    <param name="max">${PI/2}</param>
+                <param name="min">0.0</param>
+                <param name="max">${PI / 2}</param>
                 </command_interface>
-                <state_interface name="position"/>
             </joint>
         </xacro:if>
+        <!-- ros2_control Real Robot -->
         <xacro:unless value="$(arg is_sim)">
             <hardware>
                 <plugin>arduinobot_controller/ArduinobotInterface</plugin>
-                <param name = "port">/dev/ttyACM0</param>
+                <param name="port">/dev/ttyACM0</param>
             </hardware>
         </xacro:unless>
-        <hardware>
-            <plugin>gazebo_ros2_control/GazeboSystem</plugin>
-        </hardware>
         <joint name="joint_1">
             <command_interface name="position">
-                <param name="min">-${PI/2}</param>
-                <param name="max">${PI/2}</param>
+            <param name="min">-${PI / 2}</param>
+            <param name="max">${PI / 2}</param>
             </command_interface>
             <state_interface name="position"/>
@@ -35,6 +33,6 @@
         <joint name="joint_2">
             <command_interface name="position">
-                <param name="min">-${PI/2}</param>
-                <param name="max">${PI/2}</param>
+            <param name="min">-${PI / 2}</param>
+            <param name="max">${PI / 2}</param>
             </command_interface>
             <state_interface name="position"/>
@@ -42,6 +40,6 @@
         <joint name="joint_3">
             <command_interface name="position">
-                <param name="min">-${PI/2}</param>
-                <param name="max">${PI/2}</param>
+            <param name="min">-${PI / 2}</param>
+            <param name="max">${PI / 2}</param>
             </command_interface>
             <state_interface name="position"/>
@@ -49,6 +47,6 @@
         <joint name="joint_4">
             <command_interface name="position">
-                <param name="min">-${PI/2}</param>
-                <param name="max">0.0</param>
+            <param name="min">-${PI / 2}</param>
+            <param name="max">0.0</param>
             </command_interface>
             <state_interface name="position"/>
